File: pcb/eink_mahjong_compass.kicad_pcb (KiCad board)
At the start: 2 copper layers, 123.4 x 123.4 mm, 55 parts, among them J1 PH-2AWT, J2 Touch1, J3 Touch2, J4 Touch3, J5 Touch4, Q1 C10487, SW3 C318884, SW4 C318884, SW5 C318884, SW6 C318884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

Commit message: pcb: add missing trace to make deep sleep wakeup work
Connect button 4 for gpio 3 as well, so it can be used to wake up the
esp32 from deep sleep as the gpios selected for the buttons don't have
that capability.
In a future revision this should be redesigned so all buttons can act as
wakeup trigger.
Connections:
- SW6 pad 1: ESP42/BUTTON4 -> ESP3/WAKEUP
- SW6 pad 2: ESP42/BUTTON4 -> ESP3/WAKEUP
- U3 pad 15: unconnected-(U3-IO3-Pad15) -> ESP3/WAKEUP
- U3 pad 35: ESP42/BUTTON4 -> ESP3/WAKEUP
Routing:
- net ESP3/WAKEUP: track 0.00 -> 52.5 mm, vias 0 -> 3
- net ESP42/BUTTON4: track 44.2 -> 0.00 mm, vias 2 -> 0
